File: hardware/radiationsensor_r1/arrayboard_r0.brd (EAGLE design)
At the start: 160 x 100 mm, 17 parts

Commit message: final cleanup
Parts:
- removed U$1, U$10, U$11, U$12, U$13, U$14, U$15, U$16, U$2, U$3, U$4, U$5, U$6, U$7, U$8, U$9: RADIATION-SENSOR-REV1, openct:RADIATION-SENSOR-REV1
- removed U$17: ARDUINO_PRO_MINI, SparkFun-Boards:ARDUINO_PRO_MINI
- added C1: (no value), openct:0603
- added CN0, CN1, CN10, CN11, CN12, CN13, CN14, CN15, CN2, CN3, CN4, CN5, CN6, CN7, CN8, CN9: RADIATION-SENSOR-REV1, openct:RADIATION-SENSOR-REV1
- added CN16: 2524-, con-3m:PAK100/2500-24
- added CN17: 22-23-2041, con-molex:22-23-2041
- added R1: 10k, openct:0603
- added U$35, U$36, U$37, U$38: (no value), openct:MOUNT-M3
- added U1: MCP23017SS, adafruit:SSOP28
Connections:
- new net 5V: CN0.8, CN1.8, CN10.8, CN11.8, CN12.8, CN13.8, CN14.8, CN15.8, CN17.1, CN2.8, CN3.8, CN4.8, CN5.8, CN6.8, CN7.8, CN8.8, CN9.8
- new net COMP0: CN0.6, CN16.1
- new net COMP1: CN1.6, CN16.2
- new net COMP10: CN10.6, CN16.11
- new net COMP11: CN11.6, CN16.12
- new net COMP12: CN12.6, CN16.13
- new net COMP13: CN13.6, CN16.14
- new net COMP14: CN14.6, CN16.15
- new net COMP15: CN15.6, CN16.16
- new net COMP2: CN16.3, CN2.6
- new net COMP3: CN16.4, CN3.6
- new net COMP4: CN16.5, CN4.6
- new net COMP5: CN16.6, CN5.6
- new net COMP6: CN16.7, CN6.6
- new net COMP7: CN16.8, CN7.6
- new net COMP8: CN16.9, CN8.6
- new net COMP9: CN16.10, CN9.6
- new net CS0: CN0.2, U1.28
- new net CS1: CN1.2, U1.27
- new net CS10: CN10.2, U1.3
- new net CS11: CN11.2, U1.4
- new net CS12: CN12.2, U1.5
- new net CS13: CN13.2, U1.6
- new net CS14: CN14.2, U1.7
- new net CS15: CN15.2, U1.8
- new net CS2: CN2.2, U1.26
- new net CS3: CN3.2, U1.25
- new net CS4: CN4.2, U1.24
- new net CS5: CN5.2, U1.23
- new net CS6: CN6.2, U1.22
- new net CS7: CN7.2, U1.21
- new net CS8: CN8.2, U1.1
- new net CS9: CN9.2, U1.2
- new net GND: C1.2, CN0.7, CN1.7, CN10.7, CN11.7, CN12.7, CN13.7, CN14.7, CN15.7, CN16.24, CN17.2, CN17.3, CN2.7, CN3.7, CN4.7, CN5.7, CN6.7, CN7.7, CN8.7, CN9.7, U1.10, U1.15, U1.16, U1.17
- new net MOSI: CN0.4, CN1.4, CN10.4, CN11.4, CN12.4, CN13.4, CN14.4, CN15.4, CN16.20, CN2.4, CN3.4, CN4.4, CN5.4, CN6.4, CN7.4, CN8.4, CN9.4
- new net N$2: R1.2, U1.18
- new net SCL: CN16.17, U1.12
- new net SCLK: CN0.3, CN1.3, CN10.3, CN11.3, CN12.3, CN13.3, CN14.3, CN15.3, CN16.19, CN2.3, CN3.3, CN4.3, CN5.3, CN6.3, CN7.3, CN8.3, CN9.3
- new net SDA: CN16.18, U1.13
- new net VBIAS: CN0.9, CN1.9, CN10.9, CN11.9, CN12.9, CN13.9, CN14.9, CN15.9, CN17.4, CN2.9, CN3.9, CN4.9, CN5.9, CN6.9, CN7.9, CN8.9, CN9.9
- new net VLOGIC: C1.1, CN16.23, R1.1, U1.9
- new net VTEMP11: CN11.1, CN16.22
- new net VTEMP4: CN16.21, CN4.1
Routing:
- net CS1: track 0.00 -> 233.1 mm
- net CS0: track 0.00 -> 232.7 mm
- net VTEMP4: track 0.00 -> 159.1 mm
- net MOSI: track 0.00 -> 130.6 mm
- net SCLK: track 0.00 -> 130.1 mm
- net VBIAS: track 0.00 -> 119.9 mm
- net 5V: track 0.00 -> 118.7 mm
- net COMP0: track 0.00 -> 106.6 mm
- net GND: track 0.00 -> 105.1 mm, vias 0 -> 7
- net VTEMP11: track 0.00 -> 100.5 mm
- net COMP1: track 0.00 -> 99.4 mm
- net COMP2: track 0.00 -> 97.4 mm
- net COMP3: track 0.00 -> 89.9 mm
- net COMP4: track 0.00 -> 88.4 mm
- net COMP5: track 0.00 -> 80.9 mm
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- added copper zone on layer 1, net GND
- added copper zone on layer 16, net GND
Other:
- board size 160 x 100 mm -> 131.7 x 72.1 mm
- board text added: "5V"
- board text added: "GND"
- board text added: "Imaging Array Board (r0)"
- board text added: "Peter Jansen/June 2015"
- board text added: "VBIAS"
