File: hardware/radiationsensor_r1/arrayboard_r0a.brd (EAGLE design)
At the start: 160 x 100 mm, 21 parts, among them CN0 RADIATION-SENSOR-REV1, CN1 RADIATION-SENSOR-REV1, CN10 RADIATION-SENSOR-REV1, CN11 RADIATION-SENSOR-REV1, CN12 RADIATION-SENSOR-REV1, CN13 RADIATION-SENSOR-REV1, CN14 RADIATION-SENSOR-REV1, CN15 RADIATION-SENSOR-REV1, CN2 RADIATION-SENSOR-REV1, CN3 RADIATION-SENSOR-REV1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

Commit message: mechanical bits
Parts:
- added U$35, U$36, U$37, U$38: (no value), openct:MOUNT-M3
- renumbered IC1 to U1, X1 to CN16, X2 to CN17
Routing:
- net GND: vias 5 -> 7
Other:
- outline, holes or cut-outs redrawn
- board text added: "5V"
- board text added: "GND"
- board text added: "Imaging Array Board (r0)"
- board text added: "Peter Jansen/June 2015"
- board text added: "VBIAS"

Commit message: final cleanup
Other:
- board size 160 x 100 mm -> 131.7 x 72.1 mm
Changed lines of the file:
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@@
 <layer number="46" name="Milling" color="3" fill="1" visible="no" active="yes"/>
 <layer number="47" name="Measures" color="7" fill="1" visible="no" active="yes"/>
-<layer number="48" name="Document" color="7" fill="1" visible="yes" active="yes"/>
+<layer number="48" name="Document" color="14" fill="1" visible="yes" active="yes"/>
 <layer number="49" name="Reference" color="7" fill="1" visible="yes" active="yes"/>
 <layer number="50" name="dxf" color="7" fill="1" visible="no" active="no"/>
@@
 <board>
 <plain>
-<wire x1="0" y1="0" x2="160" y2="0" width="0" layer="20"/>
-<wire x1="160" y1="0" x2="160" y2="100" width="0" layer="20"/>
-<wire x1="160" y1="100" x2="0" y2="100" width="0" layer="20"/>
-<wire x1="0" y1="100" x2="0" y2="0" width="0" layer="20"/>
-<wire x1="63.5" y1="19.05" x2="63.5" y2="31.75" width="0.4064" layer="21"/>
-<wire x1="63.5" y1="31.75" x2="63.5" y2="114.3" width="0.4064" layer="21"/>
-<wire x1="63.5" y1="31.75" x2="12.7" y2="82.55" width="0.4064" layer="21"/>
-<wire x1="63.5" y1="31.75" x2="114.3" y2="82.55" width="0.4064" layer="21"/>
-<wire x1="0" y1="0" x2="127" y2="0" width="0.01" layer="21" curve="-180"/>
-<wire x1="-31.75" y1="0" x2="158.75" y2="0" width="0.4064" layer="21" curve="-180"/>
-<wire x1="-15.875" y1="0" x2="142.875" y2="0" width="0.01" layer="21" curve="-180"/>
-<wire x1="31.75" y1="31.75" x2="95.25" y2="31.75" width="0.01" layer="21" curve="-180"/>
-<wire x1="-6.35" y1="31.75" x2="133.35" y2="31.75" width="0.01" layer="21" curve="-180"/>
-<wire x1="-7.62" y1="31.75" x2="134.62" y2="31.75" width="0.01" layer="21" curve="-180"/>
-<wire x1="1.27" y1="0" x2="125.73" y2="0" width="0.01" layer="21" curve="-180"/>
-<wire x1="38.1" y1="31.75" x2="88.9" y2="31.75" width="0.01" layer="21" curve="-180"/>
+<wire x1="63.5" y1="59.75" x2="63.5" y2="91.3" width="0.4064" layer="22"/>
+<wire x1="40.25" y1="55" x2="16.95" y2="78.3" width="0.4064" layer="22"/>
+<wire x1="85" y1="53.25" x2="110.05" y2="78.3" width="0.4064" layer="22"/>
+<wire x1="0" y1="0" x2="127" y2="0" width="0.01" layer="48" curve="-180"/>
+<wire x1="-31.75" y1="0" x2="158.75" y2="0" width="0.4064" layer="48" curve="-180"/>
+<wire x1="-15.875" y1="0" x2="142.875" y2="0" width="0.01" layer="48" curve="-180"/>
+<wire x1="31.75" y1="31.75" x2="95.25" y2="31.75" width="0.01" layer="48" curve="-180"/>
+<wire x1="-6.35" y1="31.75" x2="133.35" y2="31.75" width="0.01" layer="48" curve="-180"/>
+<wire x1="-7.62" y1="31.75" x2="134.62" y2="31.75" width="0.01" layer="48" curve="-180"/>
+<wire x1="1.27" y1="0" x2="125.73" y2="0" width="0.01" layer="48" curve="-180"/>
+<wire x1="38.1" y1="31.75" x2="88.9" y2="31.75" width="0.01" layer="48" curve="-180"/>
 <wire x1="60.325" y1="60.325" x2="66.675" y2="60.325" width="0.01" layer="21"/>
-<wire x1="3.175" y1="0" x2="123.825" y2="0" width="0.254" layer="21" curve="-180"/>
-<wire x1="34.925" y1="31.75" x2="92.075" y2="31.75" width="0.254" layer="21" curve="-180"/>
+<wire x1="3.175" y1="0" x2="123.825" y2="0" width="0.254" layer="48" curve="-180"/>
+<wire x1="34.925" y1="31.75" x2="92.075" y2="31.75" width="0.254" layer="48" curve="-180"/>
 <circle x="114.3" y="44.45" radius="6.35" width="0.01" layer="20"/>
-<wire x1="87.6724" y1="58.0908" x2="84.5" y2="52.25" width="0.4064" layer="21"/>
 <circle x="114.3" y="44.45" radius="6.35" width="0.3048" layer="39"/>
 <circle x="114.3" y="44.45" radius="6.35" width="0.3048" layer="40"/>
-<circle x="12.7" y="44.45" radius="6.35" width="0.8128" layer="21"/>
+<circle x="12.7" y="44.45" radius="6.35" width="0.8128" layer="48"/>
 <circle x="114.3" y="44.45" radius="6.35" width="0.1778" layer="21"/>
 <wire x1="6" y1="71" x2="1.5" y2="63.5" width="0.01" layer="20" curve="10"/>
@@
 <circle x="114.3" y="44.45" radius="6.35" width="0.3048" layer="40"/>
 <circle x="114.3" y="44.45" radius="6.35" width="0.3048" layer="42"/>
-<wire x1="120" y1="90" x2="120" y2="10" width="0.3048" layer="21"/>
-<wire x1="10" y1="90" x2="10" y2="10" width="0.3048" layer="21"/>
 <text x="124" y="58.5" size="1.016" layer="21" rot="R315">VBIAS</text>
 <text x="118.5" y="52.75" size="1.016" layer="21" rot="R315">5V</text>
 <text x="121.25" y="54.25" size="1.016" layer="21" rot="R45">GND</text>
-<wire x1="22" y1="43.5" x2="2" y2="64.5" width="0.3048" layer="21"/>
 <text x="104.5" y="24.25" size="1.016" layer="21">Imaging Array Board (r0)</text>
 <text x="104.5" y="22.25" size="1.016" layer="21">Peter Jansen/June 2015</text>
