File: hardware/radiationsensor_r1/arrayboard_r0.sch (EAGLE design)
At the start: 17 parts

Commit message: final cleanup
Parts:
- removed U$1, U$10, U$11, U$12, U$13, U$14, U$15, U$16, U$2, U$3, U$4, U$5, U$6, U$7, U$8, U$9: RADIATION-SENSOR-REV1, openct:RADIATION-SENSOR-REV1
- removed U$17: ARDUINO_PRO_MINI, SparkFun-Boards:ARDUINO_PRO_MINI
- added C1: (no value), openct:CAP0603
- added CN0, CN1, CN10, CN11, CN12, CN13, CN14, CN15, CN2, CN3, CN4, CN5, CN6, CN7, CN8, CN9: RADIATION-SENSOR-REV1, openct:RADIATION-SENSOR-REV1
- added CN16: 2524-, con-3m:2524-
- added CN17: 22-23-2041, con-molex:22-23-2041
- added R1: 10k, openct:RESISTOR0603
- added U1: MCP23017SS, adafruit:MCP23017SS
Connections:
- new net 5V: CN0.5V, CN1.5V, CN10.5V, CN11.5V, CN12.5V, CN13.5V, CN14.5V, CN15.5V, CN17-1.S, CN2.5V, CN3.5V, CN4.5V, CN5.5V, CN6.5V, CN7.5V, CN8.5V, CN9.5V
- new net COMP0: CN0.COMP_OUT, CN16-1.KL
- new net COMP1: CN1.COMP_OUT, CN16-2.KL
- new net COMP10: CN10.COMP_OUT, CN16-11.KL
- new net COMP11: CN11.COMP_OUT, CN16-12.KL
- new net COMP12: CN12.COMP_OUT, CN16-13.KL
- new net COMP13: CN13.COMP_OUT, CN16-14.KL
- new net COMP14: CN14.COMP_OUT, CN16-15.KL
- new net COMP15: CN15.COMP_OUT, CN16-16.KL
- new net COMP2: CN16-3.KL, CN2.COMP_OUT
- new net COMP3: CN16-4.KL, CN3.COMP_OUT
- new net COMP4: CN16-5.KL, CN4.COMP_OUT
- new net COMP5: CN16-6.KL, CN5.COMP_OUT
- new net COMP6: CN16-7.KL, CN6.COMP_OUT
- new net COMP7: CN16-8.KL, CN7.COMP_OUT
- new net COMP8: CN16-9.KL, CN8.COMP_OUT
- new net COMP9: CN16-10.KL, CN9.COMP_OUT
- new net CS0: CN0.CS, U1.GPA7
- new net CS1: CN1.CS, U1.GPA6
- new net CS10: CN10.CS, U1.GPB2
- new net CS11: CN11.CS, U1.GPB3
- new net CS12: CN12.CS, U1.GPB4
- new net CS13: CN13.CS, U1.GPB5
- new net CS14: CN14.CS, U1.GPB6
- new net CS15: CN15.CS, U1.GPB7
- new net CS2: CN2.CS, U1.GPA5
- new net CS3: CN3.CS, U1.GPA4
- new net CS4: CN4.CS, U1.GPA3
- new net CS5: CN5.CS, U1.GPA2
- new net CS6: CN6.CS, U1.GPA1
- new net CS7: CN7.CS, U1.GPA0
- new net CS8: CN8.CS, U1.GPB0
- new net CS9: CN9.CS, U1.GPB1
- new net GND: C1.2, CN0.GND, CN1.GND, CN10.GND, CN11.GND, CN12.GND, CN13.GND, CN14.GND, CN15.GND, CN16-24.KL, CN17-2.S, CN17-3.S, CN2.GND, CN3.GND, CN4.GND, CN5.GND, CN6.GND, CN7.GND, CN8.GND, CN9.GND, U1.A0, U1.A1, U1.A2, U1.VSS
- new net MOSI: CN0.MOSI, CN1.MOSI, CN10.MOSI, CN11.MOSI, CN12.MOSI, CN13.MOSI, CN14.MOSI, CN15.MOSI, CN16-20.KL, CN2.MOSI, CN3.MOSI, CN4.MOSI, CN5.MOSI, CN6.MOSI, CN7.MOSI, CN8.MOSI, CN9.MOSI
- new net N$2: R1.2, U1.!RESET
- new net SCL: CN16-17.KL, U1.SCL
- new net SCLK: CN0.SCLK, CN1.SCLK, CN10.SCLK, CN11.SCLK, CN12.SCLK, CN13.SCLK, CN14.SCLK, CN15.SCLK, CN16-19.KL, CN2.SCLK, CN3.SCLK, CN4.SCLK, CN5.SCLK, CN6.SCLK, CN7.SCLK, CN8.SCLK, CN9.SCLK
- new net SDA: CN16-18.KL, U1.SDA
- new net VBIAS: CN0.VBIAS, CN1.VBIAS, CN10.VBIAS, CN11.VBIAS, CN12.VBIAS, CN13.VBIAS, CN14.VBIAS, CN15.VBIAS, CN17-4.S, CN2.VBIAS, CN3.VBIAS, CN4.VBIAS, CN5.VBIAS, CN6.VBIAS, CN7.VBIAS, CN8.VBIAS, CN9.VBIAS
- new net VLOGIC: C1.1, CN16-23.KL, R1.1, U1.VDD
- new net VTEMP11: CN11.VTEMP, CN16-22.KL
- new net VTEMP4: CN16-21.KL, CN4.VTEMP

Commit message: schematic cleanup
Other:
- note added: "ARRAY POWER CONNECTOR"
- note added: "HIGH-ENERGY PARTICLE DETECTOR ARRAY"
- note added: "IO EXPANDER"
- note added: "MICROCONTROLLER CONNECTOR"
- moved on the sheet: C1, CN16-1, CN16-10, CN16-11, CN16-12, CN16-13, CN16-14, CN16-15, CN16-16, CN16-17, CN16-18, CN16-19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
