File: hardware/radiationsensor_r1/arrayboard_r1.sch (EAGLE design)
At the start: 21 parts, among them CN0 RADIATION-SENSOR-REV1, CN1 RADIATION-SENSOR-REV1, CN10 RADIATION-SENSOR-REV1, CN11 RADIATION-SENSOR-REV1, CN12 RADIATION-SENSOR-REV1, CN13 RADIATION-SENSOR-REV1, CN14 RADIATION-SENSOR-REV1, CN15 RADIATION-SENSOR-REV1, CN16 2524-, CN17 22-23-2041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

Commit message: finished routing for imaging array board rev1
Connections:
- net 5V: now also CN17-4.S; no longer CN17-1.S
- net VBIAS: now also CN17-1.S; no longer CN17-4.S
Changed lines of the file:
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@@
 <setting verticaltext="up"/>
 </settings>
-<grid distance="0.1" unitdist="inch" unit="inch" style="lines" multiple="1" display="no" altdistance="0.01" altunitdist="inch" altunit="inch"/>
+<grid distance="0.1" unitdist="inch" unit="inch" style="lines" multiple="1" display="yes" altdistance="0.01" altunitdist="inch" altunit="inch"/>
 <layers>
 <layer number="1" name="Top" color="4" fill="1" visible="no" active="no"/>
@@
 <instance part="CN17" gate="-3" x="175.26" y="-205.74" rot="R180"/>
 <instance part="CN17" gate="-4" x="175.26" y="-203.2" rot="R180"/>
-<instance part="U$17" gate="G$1" x="182.88" y="-198.12"/>
-<instance part="U$34" gate="G$1" x="182.88" y="-215.9" rot="R180"/>
+<instance part="U$17" gate="G$1" x="182.88" y="-215.9" rot="R180"/>
+<instance part="U$34" gate="G$1" x="182.88" y="-198.12"/>
 <instance part="GND20" gate="1" x="195.58" y="-215.9"/>
 </instances>
@@
 </segment>
 <segment>
-<pinref part="CN17" gate="-1" pin="S"/>
-<wire x1="177.8" y1="-210.82" x2="182.88" y2="-210.82" width="0.1524" layer="91"/>
-<wire x1="182.88" y1="-210.82" x2="182.88" y2="-215.9" width="0.1524" layer="91"/>
+<pinref part="CN17" gate="-4" pin="S"/>
+<wire x1="177.8" y1="-203.2" x2="182.88" y2="-203.2" width="0.1524" layer="91"/>
 <pinref part="U$34" gate="G$1" pin="5V"/>
+<wire x1="182.88" y1="-203.2" x2="182.88" y2="-198.12" width="0.1524" layer="91"/>
 </segment>
 </net>
@@
 </segment>
 <segment>
-<pinref part="CN17" gate="-4" pin="S"/>
-<wire x1="177.8" y1="-203.2" x2="182.88" y2="-203.2" width="0.1524" layer="91"/>
-<wire x1="182.88" y1="-203.2" x2="182.88" y2="-198.12" width="0.1524" layer="91"/>
+<pinref part="CN17" gate="-1" pin="S"/>
+<wire x1="177.8" y1="-210.82" x2="182.88" y2="-210.82" width="0.1524" layer="91"/>
 <pinref part="U$17" gate="G$1" pin="VBIAS"/>
+<wire x1="182.88" y1="-210.82" x2="182.88" y2="-215.9" width="0.1524" layer="91"/>
 </segment>
 </net>
